File: pcb/left/left.kicad_pcb (KiCad board)
At the start: 2 copper layers, 138.1 x 116.7 mm, 87 parts, among them J1 78171-0004, J2 78171-0004, J3 AVR-ISP-6, SW1 SW_Reset, U1 ATmega32U4-A, Y1 16mHz

Commit message: Update pcbs
Parts:
- added R4: 4.7kΩ, Resistor_SMD:R_0603_1608Metric, B.Cu at (133.6, 144.2)
- added R5: 4.7kΩ, Resistor_SMD:R_0603_1608Metric, B.Cu at (132.0, 145.4)
- added R6: 10kΩ, Resistor_SMD:R_0603_1608Metric, B.Cu at (147.0, 148.0)
- moved J2 0.10 mm to (83.5, 144.4)
Connections:
- J1 pad MP: (no net) -> GND
- J2 pad MP: (no net) -> GND
- J3 pad 3: SCL -> SCK
- U1 pad 18: Col3 -> SCL
- U1 pad 32: unconnected-(U1-PC7-Pad32) -> Col3
- U1 pad 41: unconnected-(U1-PF0-Pad41) -> Net-(U1-PF0)
- U1 pad 9: SCL -> SCK
Routing:
- net SCK: track 0.00 -> 88.6 mm, vias 0 -> 3
- net +5V: track 144.7 -> 216.2 mm
- net Col3: track 137.0 -> 154.4 mm, vias 0 -> 2
- net GND: track 28.9 -> 23.3 mm
- net SDA: track 81.8 -> 86.6 mm, vias 2 -> 3
- net RESET: track 109.3 -> 113.2 mm
- net Col0: track 234.6 -> 238.4 mm
- net SCL: track 90.1 -> 87.8 mm
- net Net-(U1-PF0): track 0.00 -> 2.01 mm
- net Col2: track 155.6 -> 156.2 mm
Other:
- board size 138.1 x 116.7 mm -> 138.1 x 114.3 mm
