File: pcb/pad/encoder_daughterboard/encoder_daughterboard.kicad_sch (KiCad schematic)
At the start: 9 parts, among them J1 Conn_01x12, SW1 RotaryEncoder_Switch_MP, SW2 RotaryEncoder_Switch_MP, SW3 RotaryEncoder_Switch_MP

Commit message: Update encoder_daughterboard
Parts:
- J1: value Conn_01x12 -> AFA07-S12FCA-00; LCSC Part Number (none) -> C262718
- SW1, SW2, SW3: value RotaryEncoder_Switch_MP -> EC11E09244BS
Connections:
- net BCol0: no longer J1.8 (Pin_8)
- net BCol1: no longer J1.9 (Pin_9)
- net BCol2: now also J1.1 (Pin_1); no longer J1.10 (Pin_10)
- net BRow0: no longer J1.11 (Pin_11)
- net E0A: no longer J1.2 (Pin_2)
- net E0B: no longer J1.1 (Pin_1)
- net E1A: no longer J1.4 (Pin_4)
- net E1B: no longer J1.3 (Pin_3)
- net E2A: no longer J1.5 (Pin_5)
- net E2B: no longer J1.6 (Pin_6)
- net GND: no longer J1.12 (Pin_12), J1.7 (Pin_7)
Changed lines of the file:
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@@
 	(global_label "E2A"
 		(shape input)
-		(at 215.9 81.28 180)
+		(at 199.39 81.28 180)
 		(fields_autoplaced yes)
 		(effects
@@
 		)
 		(property "Intersheetrefs" "${INTERSHEET_REFS}"
-			(at 212.0404 81.28 0)
+			(at 195.5304 81.28 0)
 			(effects
 				(font
@@
 	(global_label "E0A"
 		(shape input)
-		(at 215.9 73.66 180)
+		(at 199.39 73.66 180)
 		(fields_autoplaced yes)
 		(effects
@@
 		)
 		(property "Intersheetrefs" "${INTERSHEET_REFS}"
-			(at 212.0404 73.66 0)
+			(at 195.5304 73.66 0)
 			(effects
 				(font
@@
 	(global_label "BCol2"
 		(shape output)
-		(at 215.9 93.98 180)
+		(at 215.9 71.12 180)
 		(fields_autoplaced yes)
 		(effects
@@
 		)
 		(property "Intersheetrefs" "${INTERSHEET_REFS}"
-			(at 210.7704 93.98 0)
+			(at 210.7704 71.12 0)
 			(effects
 				(font
@@
 	(global_label "E0B"
 		(shape input)
-		(at 215.9 71.12 180)
+		(at 199.39 71.12 180)
 		(fields_autoplaced yes)
 		(effects
@@
 		)
 		(property "Intersheetrefs" "${INTERSHEET_REFS}"
-			(at 211.9315 71.12 0)
+			(at 195.4215 71.12 0)
 			(effects
 				(font
@@
 	(global_label "E2B"
 		(shape input)
-		(at 215.9 83.82 180)
+		(at 199.39 83.82 180)
 		(fields_autoplaced yes)
 		(effects
@@
 		)
 		(property "Intersheetrefs" "${INTERSHEET_REFS}"
-			(at 211.9315 83.82 0)
+			(at 195.4215 83.82 0)
 			(effects
 				(font
@@
 	(global_label "BRow0"
 		(shape input)
-		(at 215.9 96.52 180)
+		(at 199.39 96.52 180)
 		(fields_autoplaced yes)
 		(effects
@@
 		)
 		(property "Intersheetrefs" "${INTERSHEET_REFS}"
-			(at 210.3712 96.52 0)
+			(at 193.8612 96.52 0)
 			(effects
 				(font
@@
 	(global_label "BCol0"
 		(shape output)
-		(at 215.9 88.9 180)
+		(at 199.39 88.9 180)
 		(fields_autoplaced yes)
 		(effects
@@
 		)
 		(property "Intersheetrefs" "${INTERSHEET_REFS}"
-			(at 210.7704 88.9 0)
+			(at 194.2604 88.9 0)
 			(effects
 				(font
@@
 	(global_label "BCol1"
 		(shape output)
-		(at 215.9 91.44 180)
+		(at 199.39 91.44 180)
 		(fields_autoplaced yes)
 		(effects
@@
 		)
 		(property "Intersheetrefs" "${INTERSHEET_REFS}"
-			(at 210.7704 91.44 0)
+			(at 194.2604 91.44 0)
 			(effects
 				(font
@@
 	(global_label "E1B"
 		(shape input)
-		(at 215.9 76.2 180)
+		(at 199.39 76.2 180)
 		(fields_autoplaced yes)
 		(effects
@@
 		)
 		(property "Intersheetrefs" "${INTERSHEET_REFS}"
-			(at 211.9315 76.2 0)
+			(at 195.4215 76.2 0)
 			(effects
 				(font
@@
 	(global_label "E1A"
 		(shape input)
-		(at 215.9 78.74 180)
+		(at 199.39 78.74 180)
 		(fields_autoplaced yes)
 		(effects
@@
 		)
 		(property "Intersheetrefs" "${INTERSHEET_REFS}"
-			(at 212.0404 78.74 0)
+			(at 195.5304 78.74 0)
 			(effects
 				(font
@@
 	(symbol
 		(lib_id "power:GND")
-		(at 215.9 99.06 270)
+		(at 199.39 99.06 270)
 		(unit 1)
 		(exclude_from_sim no)
@@
 		(fields_autoplaced yes)
 		(property "Reference" "#PWR07"
-			(at 209.55 99.06 0)
+			(at 193.04 99.06 0)
 			(effects
 				(font
@@
 		)
 		(property "Value" "GND"
-			(at 212.09 99.0599 90)
+			(at 195.58 99.0599 90)
 			(effects
 				(font
@@
 		)
 		(property "Footprint" ""
-			(at 215.9 99.06 0)
+			(at 199.39 99.06 0)
 			(effects
 				(font
@@
 		)
 		(property "Datasheet" ""
-			(at 215.9 99.06 0)
+			(at 199.39 99.06 0)
 			(effects
 				(font
@@
 		)
 		(property "Description" "Power symbol creates a global label with name \"GND\" , ground"
-			(at 215.9 99.06 0)
+			(at 199.39 99.06 0)
 			(effects
 				(font
@@
 			)
 		)
-		(property "Value" "Conn_01x12"
+		(property "Value" "AFA07-S12FCA-00"
 			(at 223.52 86.7155 0)
 			(effects
@@
 			)
 		)
+		(property "LCSC Part Number" "C262718"
+			(at 220.98 83.82 0)
+			(effects
+				(font
+					(size 1.27 1.27)
+				)
+				(hide yes)
+			)
+		)
 		(pin "7"
 		)
@@
 			)
 		)
-		(property "Value" "RotaryEncoder_Switch_MP"
+		(property "Value" "EC11E09244BS"
 			(at 165.1 74.93 0)
 			(effects
@@
 			)
 		)
-		(property "Value" "RotaryEncoder_Switch_MP"
+		(property "Value" "EC11E09244BS"
 			(at 125.73 74.93 0)
 			(effects
@@
 	(symbol
 		(lib_id "power:GND")
-		(at 215.9 86.36 270)
+		(at 199.39 86.36 270)
 		(unit 1)
 		(exclude_from_sim no)
@@
 		(fields_autoplaced yes)
 		(property "Reference" "#PWR08"
-			(at 209.55 86.36 0)
+			(at 193.04 86.36 0)
 			(effects
 				(font
@@
 		)
 		(property "Value" "GND"
-			(at 212.09 86.3599 90)
+			(at 195.58 86.3599 90)
 			(effects
 				(font
@@
 		)
 		(property "Footprint" ""
-			(at 215.9 86.36 0)
+			(at 199.39 86.36 0)
 			(effects
 				(font
@@
 		)
 		(property "Datasheet" ""
-			(at 215.9 86.36 0)
+			(at 199.39 86.36 0)
 			(effects
 				(font
@@
 		)
 		(property "Description" "Power symbol creates a global label with name \"GND\" , ground"
-			(at 215.9 86.36 0)
+			(at 199.39 86.36 0)
 			(effects
 				(font
@@
 			)
 		)
-		(property "Value" "RotaryEncoder_Switch_MP"
+		(property "Value" "EC11E09244BS"
 			(at 88.9 74.93 0)
 			(effects

Commit message: Update encoder_daughterboard
Parts:
- removed H1: MountingHole_Pad_MP, MountingHole:MountingHole_3.2mm_M3_DIN965_Pad_TopOnly, symbol Mechanical:MountingHole_Pad_MP
- added H1: MountingHole_Pad, MountingHole:MountingHole_3.2mm_M3_DIN965_Pad_TopOnly, symbol Mechanical:MountingHole_Pad
Connections:
- net BCol0: now also J1.10 (Pin_10)
- net BCol1: now also J1.7 (Pin_7)
- net BRow0: now also J1.4 (Pin_4)
- net E0A: now also J1.11 (Pin_11)
- net E0B: now also J1.12 (Pin_12)
- net E1A: now also J1.5 (Pin_5)
- net E1B: now also J1.6 (Pin_6)
- net E2A: now also J1.3 (Pin_3)
- net E2B: now also J1.2 (Pin_2)
- net GND: now also J1.8 (Pin_8), J1.9 (Pin_9), H1.1

Commit message: Update FPC connectors
Parts:
- J1: footprint Connector_FFC-FPC:JUSHUO_AFA07-S12FCA-00_1x12-1MP_P1.0mm_Horizontal -> Connector_FFC-FPC:Hirose_FH12-12S-0.5SH_1x12-1MP_P0.50mm_Horizontal
Changed lines of the file:
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@@
 			)
 		)
-		(property "Footprint" "Connector_FFC-FPC:JUSHUO_AFA07-S12FCA-00_1x12-1MP_P1.0mm_Horizontal"
+		(property "Footprint" "Connector_FFC-FPC:Hirose_FH12-12S-0.5SH_1x12-1MP_P0.50mm_Horizontal"
 			(at 220.98 83.82 0)
 			(effects
